File: ControlBoard/Control Board.kicad_pcb (KiCad board)
At the start: 2 copper layers, 120.7 x 77.5 mm, 57 parts, among them J1 Conn_01x02_Pin, Q1 BSS138, U1 SN74LVC245APW, U2 ULN2003

Commit message: Update to Control Board
Other:
- board text added: "TODO: Need voltage divider + pullup on the !shutdown turns out this is a floating input"
